File: kicad/frequency_counter.kicad_sch (KiCad schematic)
At the start: 27 parts, among them J101 SMA, J102 SMA, J103 USB-C, J104 DISPLAY, SW1 SW_SPST, SW103 SPST, SW2 SW_SPST

Commit message: finish 2.0 part selection
Parts:
- BT101: footprint Connector_Wire:SolderWire-0.5sqmm_1x02_P4.6mm_D0.9mm_OD2.1mm -> Connector_JST:JST_ZH_B2B-ZR_1x02_P1.50mm_Vertical; Supplier Generic -> (none)
- R105, R106: footprint (none) -> Custom:R_0402_1005Metric_Fix; MPN (none) -> RC0402JR-074K7L
- SW1, SW2: value SW_SPST -> PushBtn; footprint (none) -> Button_Switch_SMD:SW_Push_1P1T_NO_E-Switch_TL3301NxxxxxG; MPN (none) -> 2-1977223-4
- SW103: value SPST -> Rocker
- TP101, TP102: MPN (none) -> RCWCTE; Supplier https://www.digikey.com/en/products/detail/harwin-inc/S2751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 -> (none)
Changed lines of the file:
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@@
 	(title_block
 		(title "Frequency Counter")
-		(date "2026-02-17")
+		(date "2026-02-18")
 		(rev "2.0-draft")
 		(company "vladaviedov.org")
@@
 			)
 		)
-		(property "Supplier" ""
-			(at 20.32 52.07 0)
-			(effects
-				(font
-					(size 1.27 1.27)
-				)
-				(hide yes)
-			)
-		)
 		(property "MPN" "CON-SMA-EDGE-S"
 			(at 20.32 52.07 0)
@@
 			)
 		)
-		(property "Value" "SW_SPST"
+		(property "Value" "PushBtn"
 			(at 177.8 68.58 0)
 			(effects
@@
 			)
 		)
-		(property "Footprint" ""
+		(property "Footprint" "Button_Switch_SMD:SW_Push_1P1T_NO_E-Switch_TL3301NxxxxxG"
 			(at 177.8 72.39 0)
 			(effects
@@
 			)
 		)
+		(property "MPN" "2-1977223-4 "
+			(at 177.8 72.39 0)
+			(effects
+				(font
+					(size 1.27 1.27)
+				)
+				(hide yes)
+			)
+		)
 		(pin "2"
 		)
@@
 			)
 		)
-		(property "Supplier" ""
-			(at 67.31 182.88 0)
-			(effects
-				(font
-					(size 1.27 1.27)
-				)
-				(hide yes)
-			)
-		)
 		(property "MPN" "RC0402JR-135K1L"
 			(at 67.31 182.88 0)
@@
 			)
 		)
-		(property "Supplier" ""
-			(at 20.32 27.94 0)
-			(effects
-				(font
-					(size 1.27 1.27)
-				)
-				(hide yes)
-			)
-		)
 		(property "MPN" "CON-SMA-EDGE-S"
 			(at 20.32 27.94 0)
@@
 			)
 		)
-		(property "Supplier" ""
-			(at 76.2 96.52 0)
-			(effects
-				(font
-					(size 1.27 1.27)
-				)
-				(hide yes)
-			)
-		)
 		(pin "3"
 		)
@@
 			)
 		)
-		(property "Supplier" ""
-			(at 163.83 107.95 90)
-			(effects
-				(font
-					(size 1.27 1.27)
-				)
-				(hide yes)
-			)
-		)
 		(property "MPN" "B1911UY--20D000114U1930"
 			(at 163.83 107.95 90)
@@
 			)
 		)
-		(property "Value" "SPST"
+		(property "Value" "Rocker"
 			(at 35.56 125.73 0)
 			(effects
@@
 			)
 		)
-		(property "Footprint" ""
+		(property "Footprint" "Custom:R_0402_1005Metric_Fix"
 			(at 93.726 92.964 90)
 			(effects
@@
 			)
 		)
+		(property "MPN" "RC0402JR-074K7L"
+			(at 92.71 92.71 0)
+			(effects
+				(font
+					(size 1.27 1.27)
+				)
+				(hide yes)
+			)
+		)
 		(pin "2"
 		)
@@
 			)
 		)
-		(property "Supplier" ""
-			(at 179.07 97.79 0)
-			(effects
-				(font
-					(size 1.27 1.27)
-				)
-				(hide yes)
-			)
-		)
 		(property "MPN" "RC0402JR-13220RL"
 			(at 179.07 97.79 0)
@@
 			)
 		)
-		(property "Supplier" ""
-			(at 54.61 182.88 0)
-			(effects
-				(font
-					(size 1.27 1.27)
-				)
-				(hide yes)
-			)
-		)
 		(property "MPN" "RC0402JR-135K1L"
 			(at 54.61 182.88 0)
@@
 			)
 		)
-		(property "Supplier" ""
-			(at 36.83 168.91 0)
-			(effects
-				(font
-					(size 1.27 1.27)
-				)
-				(hide yes)
-			)
-		)
 		(property "MPN" "USB4125-GF-A"
 			(at 36.83 168.91 0)
@@
 			)
 		)
-		(property "Supplier" ""
-			(at 179.07 107.95 90)
-			(effects
-				(font
-					(size 1.27 1.27)
-				)
-				(hide yes)
-			)
-		)
 		(property "MPN" "B1911NG--20D000214U1930"
 			(at 179.07 107.95 90)
@@
 			)
 		)
-		(property "Supplier" "https://www.digikey.com/en/products/detail/harwin-inc/S2751-46R/5250499?s=N4IgTCBcDaIJwFYwFowDY0BZkEZkDsATEAXQF8g"
+		(property "MPN" "RCWCTE"
 			(at 67.31 45.72 90)
 			(effects
@@
 			)
 		)
-		(property "Footprint" ""
+		(property "Footprint" "Custom:R_0402_1005Metric_Fix"
 			(at 105.156 92.964 90)
 			(effects
@@
 			)
 		)
+		(property "MPN" "RC0402JR-074K7L"
+			(at 104.14 92.71 0)
+			(effects
+				(font
+					(size 1.27 1.27)
+				)
+				(hide yes)
+			)
+		)
 		(pin "2"
 		)
@@
 			)
 		)
-		(property "Supplier" "https://www.digikey.com/en/products/detail/harwin-inc/S2751-46R/5250499?s=N4IgTCBcDaIJwFYwFowDY0BZkEZkDsATEAXQF8g"
+		(property "MPN" "RCWCTE"
 			(at 16.51 127 0)
 			(effects
@@
 			)
 		)
-		(property "Supplier" ""
-			(at 163.83 97.79 0)
-			(effects
-				(font
-					(size 1.27 1.27)
-				)
-				(hide yes)
-			)
-		)
 		(property "MPN" "RC0402JR-13220RL"
 			(at 163.83 97.79 0)
@@
 			)
 		)
-		(property "Footprint" "Connector_Wire:SolderWire-0.5sqmm_1x02_P4.6mm_D0.9mm_OD2.1mm"
+		(property "Footprint" "Connector_JST:JST_ZH_B2B-ZR_1x02_P1.50mm_Vertical"
 			(at 26.67 138.176 90)
 			(effects
@@
 			)
 		)
-		(property "Supplier" "Generic"
-			(at 26.67 139.7 0)
-			(effects
-				(font
-					(size 1.27 1.27)
-				)
-				(hide yes)
-			)
-		)
 		(property "Sim.Device" "V"
 			(at 26.67 139.7 0)
@@
 			)
 		)
-		(property "Value" "SW_SPST"
+		(property "Value" "PushBtn"
 			(at 177.8 78.74 0)
 			(effects
@@
 			)
 		)
-		(property "Footprint" ""
+		(property "Footprint" "Button_Switch_SMD:SW_Push_1P1T_NO_E-Switch_TL3301NxxxxxG"
 			(at 177.8 82.55 0)
 			(effects
@@
 			)
 		)
+		(property "MPN" "2-1977223-4 "
+			(at 177.8 82.55 0)
+			(effects
+				(font
+					(size 1.27 1.27)
+				)
+				(hide yes)
+			)
+		)
 		(pin "2"
 		)
@@
 			(at 233.68 102.87 0)
 			(effects
-				(font
-					(size 1.27 1.27)
-				)
-				(hide yes)
-			)
-		)
-		(property "Supplier" ""
-			(at 233.68 102.87 0)
-			(effects
