File: kicad/frequency_counter.kicad_sch (KiCad schematic)
At the start: 27 parts, among them J101 SMA, J102 SMA, J103 USB-C, J104 DISPLAY, SW1 PushBtn, SW103 Rocker, SW2 PushBtn

Commit message: assign references
Parts:
- TP101: renamed from TP102; value TestPoint -> RCW
- TP102: renamed from TP101; value TestPoint -> RCW
- renumbered H105 to H102, H102 to H103, H106 to H104, H103 to H105, H107 to H106, H104 to H107, J104 to J103, J103 to J104, R106 to R101, R105 to R102, R101 to R105, R102 to R106, SW1 to SW101, SW2 to SW102
Changed lines of the file:
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@@
 		(dnp no)
 		(fields_autoplaced yes)
-		(property "Reference" "#PWR0107"
+		(property "Reference" "#PWR0106"
 			(at 83.82 87.63 0)
 			(effects
@@
 			(project ""
 				(path "/62339e8b-4e00-440f-8d81-4472a4f50c26"
-					(reference "#PWR0107")
+					(reference "#PWR0106")
 					(unit 1)
 				)
@@
 		(dnp no)
 		(fields_autoplaced yes)
-		(property "Reference" "SW1"
+		(property "Reference" "SW101"
 			(at 177.8 66.04 0)
 			(effects
@@
 			(project ""
 				(path "/62339e8b-4e00-440f-8d81-4472a4f50c26"
-					(reference "SW1")
+					(reference "SW101")
 					(unit 1)
 				)
@@
 		(dnp no)
 		(fields_autoplaced yes)
-		(property "Reference" "R102"
+		(property "Reference" "R106"
 			(at 69.85 181.6099 0)
 			(effects
@@
 			(project "frequency_counter"
 				(path "/62339e8b-4e00-440f-8d81-4472a4f50c26"
-					(reference "R102")
+					(reference "R106")
 					(unit 1)
 				)
@@
 		(dnp no)
 		(fields_autoplaced yes)
-		(property "Reference" "J104"
+		(property "Reference" "J103"
 			(at 76.835 88.9 0)
 			(effects
@@
 			(project ""
 				(path "/62339e8b-4e00-440f-8d81-4472a4f50c26"
-					(reference "J104")
+					(reference "J103")
 					(unit 1)
 				)
@@
 		(dnp no)
 		(fields_autoplaced yes)
-		(property "Reference" "H105"
+		(property "Reference" "H102"
 			(at 218.44 152.3999 0)
 			(effects
@@
 			(project "frequency_counter"
 				(path "/62339e8b-4e00-440f-8d81-4472a4f50c26"
-					(reference "H105")
+					(reference "H102")
 					(unit 1)
 				)
@@
 		(dnp no)
 		(fields_autoplaced yes)
-		(property "Reference" "#PWR0109"
+		(property "Reference" "#PWR0108"
 			(at 163.83 120.65 0)
 			(effects
@@
 			(project ""
 				(path "/62339e8b-4e00-440f-8d81-4472a4f50c26"
-					(reference "#PWR0109")
+					(reference "#PWR0108")
 					(unit 1)
 				)
@@
 		(dnp no)
 		(fields_autoplaced yes)
-		(property "Reference" "H103"
+		(property "Reference" "H105"
 			(at 243.84 130.8099 0)
 			(effects
@@
 			(project "frequency_counter"
 				(path "/62339e8b-4e00-440f-8d81-4472a4f50c26"
-					(reference "H103")
+					(reference "H105")
 					(unit 1)
 				)
@@
 		(dnp no)
 		(fields_autoplaced yes)
-		(property "Reference" "H106"
+		(property "Reference" "H104"
 			(at 231.14 152.3999 0)
 			(effects
@@
 			(project "frequency_counter"
 				(path "/62339e8b-4e00-440f-8d81-4472a4f50c26"
-					(reference "H106")
+					(reference "H104")
 					(unit 1)
 				)
@@
 		(dnp no)
 		(fields_autoplaced yes)
-		(property "Reference" "#PWR0112"
+		(property "Reference" "#PWR0109"
 			(at 179.07 120.65 0)
 			(effects
@@
 			(project "frequency_counter"
 				(path "/62339e8b-4e00-440f-8d81-4472a4f50c26"
-					(reference "#PWR0112")
+					(reference "#PWR0109")
 					(unit 1)
 				)
@@
 		(dnp no)
 		(fields_autoplaced yes)
-		(property "Reference" "R106"
+		(property "Reference" "R101"
 			(at 95.25 91.4399 0)
 			(effects
@@
 			(project "frequency_counter"
 				(path "/62339e8b-4e00-440f-8d81-4472a4f50c26"
-					(reference "R106")
+					(reference "R101")
 					(unit 1)
 				)
@@
 		(dnp no)
 		(fields_autoplaced yes)
-		(property "Reference" "#PWR01"
+		(property "Reference" "#PWR0102"
 			(at 20.32 66.04 0)
 			(effects
@@
 			(project "frequency_counter"
 				(path "/62339e8b-4e00-440f-8d81-4472a4f50c26"
-					(reference "#PWR01")
+					(reference "#PWR0102")
 					(unit 1)
 				)
@@
 		(dnp no)
 		(fields_autoplaced yes)
-		(property "Reference" "H107"
+		(property "Reference" "H106"
 			(at 243.84 152.3999 0)
 			(effects
@@
 			(project "frequency_counter"
 				(path "/62339e8b-4e00-440f-8d81-4472a4f50c26"
-					(reference "H107")
+					(reference "H106")
 					(unit 1)
 				)
@@
 		(dnp no)
 		(fields_autoplaced yes)
-		(property "Reference" "R101"
+		(property "Reference" "R105"
 			(at 57.15 181.6099 0)
 			(effects
@@
 			(project ""
 				(path "/62339e8b-4e00-440f-8d81-4472a4f50c26"
-					(reference "R101")
+					(reference "R105")
 					(unit 1)
 				)
@@
 		(dnp no)
 		(fields_autoplaced yes)
-		(property "Reference" "J103"
+		(property "Reference" "J104"
 			(at 36.83 151.13 0)
 			(effects
@@
 			(project ""
 				(path "/62339e8b-4e00-440f-8d81-4472a4f50c26"
-					(reference "J103")
+					(reference "J104")
 					(unit 1)
 				)
@@
 		(dnp no)
 		(fields_autoplaced yes)
-		(property "Reference" "TP102"
+		(property "Reference" "TP101"
 			(at 64.008 40.64 90)
 			(effects
@@
 			)
 		)
-		(property "Value" "TestPoint"
+		(property "Value" "RCW"
 			(at 64.008 43.18 90)
 			(effects
@@
 			(project "frequency_counter"
 				(path "/62339e8b-4e00-440f-8d81-4472a4f50c26"
-					(reference "TP102")
+					(reference "TP101")
 					(unit 1)
 				)
@@
 		(dnp no)
 		(fields_autoplaced yes)
-		(property "Reference" "R105"
+		(property "Reference" "R102"
 			(at 106.68 91.4399 0)
 			(effects
@@
 			(project ""
 				(path "/62339e8b-4e00-440f-8d81-4472a4f50c26"
-					(reference "R105")
+					(reference "R102")
 					(unit 1)
 				)
@@
 		(dnp no)
 		(fields_autoplaced yes)
-		(property "Reference" "H104"
+		(property "Reference" "H107"
 			(at 256.54 130.8099 0)
 			(effects
@@
 			(project "frequency_counter"
 				(path "/62339e8b-4e00-440f-8d81-4472a4f50c26"
-					(reference "H104")
+					(reference "H107")
 					(unit 1)
 				)
@@
 		(dnp no)
 		(fields_autoplaced yes)
-		(property "Reference" "TP101"
+		(property "Reference" "TP102"
 			(at 19.05 122.4279 0)
 			(effects
@@
 			)
 		)
-		(property "Value" "TestPoint"
+		(property "Value" "RCW"
 			(at 19.05 124.9679 0)
 			(effects
@@
 			(project "frequency_counter"
 				(path "/62339e8b-4e00-440f-8d81-4472a4f50c26"
-					(reference "TP101")
+					(reference "TP102")
 					(unit 1)
 				)
@@
 		(dnp no)
 		(fields_autoplaced yes)
-		(property "Reference" "H102"
+		(property "Reference" "H103"
 			(at 231.14 130.8099 0)
 			(effects
@@
 			(project "frequency_counter"
 				(path "/62339e8b-4e00-440f-8d81-4472a4f50c26"
-					(reference "H102")
+					(reference "H103")
 					(unit 1)
 				)
@@
 		(on_board yes)
 		(dnp no)
-		(property "Reference" "#PWR0116"
+		(property "Reference" "#PWR0112"
 			(at 215.9 168.91 0)
 			(effects
@@
 			(project "frequency_counter"
 				(path "/62339e8b-4e00-440f-8d81-4472a4f50c26"
-					(reference "#PWR0116")
+					(reference "#PWR0112")
 					(unit 1)
 				)
@@
 		(dnp no)
 		(fields_autoplaced yes)
-		(property "Reference" "SW2"
+		(property "Reference" "SW102"
 			(at 177.8 76.2 0)
 			(effects
@@
 			(project "frequency_counter"
 				(path "/62339e8b-4e00-440f-8d81-4472a4f50c26"
-					(reference "SW2")
+					(reference "SW102")
 					(unit 1)
 				)
@@
 		(dnp no)
 		(fields_autoplaced yes)
-		(property "Reference" "#PWR04"
+		(property "Reference" "#PWR0110"
 			(at 185.42 91.44 0)
 			(effects
@@
 			(project ""
 				(path "/62339e8b-4e00-440f-8d81-4472a4f50c26"
-					(reference "#PWR04")
+					(reference "#PWR0110")
 					(unit 1)
 				)
@@
 		(on_board yes)
 		(dnp no)
-		(property "Reference" "#PWR0108"
+		(property "Reference" "#PWR0107"
 			(at 86.36 110.49 0)
 			(effects
@@
 			(project ""
 				(path "/62339e8b-4e00-440f-8d81-4472a4f50c26"
-					(reference "#PWR0108")
+					(reference "#PWR0107")
 					(unit 1)
 				)
@@
 		(dnp no)
 		(fields_autoplaced yes)
-		(property "Reference" "#PWR0115"
+		(property "Reference" "#PWR0113"
 			(at 233.68 121.92 0)
 			(effects
@@
 			(project ""
 				(path "/62339e8b-4e00-440f-8d81-4472a4f50c26"
-					(reference "#PWR0115")
+					(reference "#PWR0113")
 					(unit 1)
 				)
@@
 		(on_board yes)
 		(dnp no)
-		(property "Reference" "#PWR0114"
+		(property "Reference" "#PWR0111"
 			(at 215.9 147.32 0)
 			(effects
@@
 			(project ""
 				(path "/62339e8b-4e00-440f-8d81-4472a4f50c26"
-					(reference "#PWR0114")
-					(unit 1)
-				)
+					(reference "#PWR0111")
+					(unit 1)
+				)

Commit message: minor fixes, 2.0 schematic
Parts:
- TP101, TP102: footprint Custom:TestPoint_Pad_2.0x2.0mm_Fix -> Custom:TestPoint_KOA_RCW
Changed lines of the file:
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@@
 	(title_block
 		(title "Frequency Counter")
-		(date "2026-02-18")
-		(rev "2.0-draft")
+		(date "2026-02-19")
+		(rev "2.0")
 		(company "vladaviedov.org")
 		(comment 1 "Maximum Precision (125 mHz ~ 325 MHz): 62.5 mHz")
@@
 			)
 		)
-		(property "Footprint" "Custom:TestPoint_Pad_2.0x2.0mm_Fix"
+		(property "Footprint" "Custom:TestPoint_KOA_RCW"
 			(at 67.31 40.64 0)
 			(effects
@@
 			)
 		)
-		(property "Footprint" "Custom:TestPoint_Pad_2.0x2.0mm_Fix"
+		(property "Footprint" "Custom:TestPoint_KOA_RCW"
 			(at 21.59 127 0)
 			(effects

Commit message: redesign pcb for 2.0
Parts:
- renumbered H103 to H102, H105 to H103, H107 to H104, H102 to H105, H104 to H106, H106 to H107
Changed lines of the file:
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@@
 		(dnp no)
 		(fields_autoplaced yes)
-		(property "Reference" "H102"
+		(property "Reference" "H105"
 			(at 218.44 152.3999 0)
 			(effects
@@
 			(project "frequency_counter"
 				(path "/62339e8b-4e00-440f-8d81-4472a4f50c26"
-					(reference "H102")
+					(reference "H105")
 					(unit 1)
 				)
@@
 		(dnp no)
 		(fields_autoplaced yes)
-		(property "Reference" "H105"
+		(property "Reference" "H103"
 			(at 243.84 130.8099 0)
 			(effects
@@
 			(project "frequency_counter"
 				(path "/62339e8b-4e00-440f-8d81-4472a4f50c26"
-					(reference "H105")
+					(reference "H103")
 					(unit 1)
 				)
@@
 		(dnp no)
 		(fields_autoplaced yes)
-		(property "Reference" "H104"
+		(property "Reference" "H106"
 			(at 231.14 152.3999 0)
 			(effects
@@
 			(project "frequency_counter"
 				(path "/62339e8b-4e00-440f-8d81-4472a4f50c26"
-					(reference "H104")
+					(reference "H106")
 					(unit 1)
 				)
@@
 		(dnp no)
 		(fields_autoplaced yes)
-		(property "Reference" "H106"
+		(property "Reference" "H107"
 			(at 243.84 152.3999 0)
 			(effects
@@
 			(project "frequency_counter"
 				(path "/62339e8b-4e00-440f-8d81-4472a4f50c26"
-					(reference "H106")
+					(reference "H107")
 					(unit 1)
 				)
@@
 		(dnp no)
 		(fields_autoplaced yes)
-		(property "Reference" "H107"
+		(property "Reference" "H104"
 			(at 256.54 130.8099 0)
 			(effects
@@
 			(project "frequency_counter"
 				(path "/62339e8b-4e00-440f-8d81-4472a4f50c26"
-					(reference "H107")
+					(reference "H104")
 					(unit 1)
 				)
@@
 		(dnp no)
 		(fields_autoplaced yes)
-		(property "Reference" "H103"
+		(property "Reference" "H102"
 			(at 231.14 130.8099 0)
 			(effects
@@
 			(project "frequency_counter"
 				(path "/62339e8b-4e00-440f-8d81-4472a4f50c26"
-					(reference "H103")
-					(unit 1)
-				)
+					(reference "H102")
+					(unit 1)
+				)
