File: kicad/frontend.kicad_sch (KiCad schematic)
At the start: 26 parts, among them U1 NCS2250, U201 TLV3603DCK

Commit message: replace alum caps with ceramics, change mpn labeling
Parts:
- CD1: MPN (none) -> KGM05AR51C104KH; Supplier https://www.digikey.com/en/products/detail/kyocera-avx/KGM0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 -> (none)
- CD201: MPN (none) -> CC0402JRNPO9BN101; Supplier https://www.digikey.com/en/products/detail/yageo/CC0402JRNP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 -> (none)
- CD202: MPN (none) -> GRM155R71C103KA01D; Supplier https://www.digikey.com/en/products/detail/murata-electroni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 -> (none)
- CD203: MPN (none) -> 0402ZD105KAT2A; Supplier https://www.digikey.com/en/products/detail/kyocera-avx/0402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 -> (none)
- D1, D2, D201, D202, D3, D4, D5, D6: MPN (none) -> SMP1345-040LF; Supplier https://www.digikey.com/en/products/detail/skyworks-solutio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 -> (none)
- D203: MPN (none) -> RBE01VYM6AFHTR; Supplier https://www.digikey.com/en/products/detail/rohm-semiconduct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 -> (none)
- R2: MPN (none) -> RC0402JR-071KL; Supplier https://www.digikey.com/en/products/detail/yageo/RC0402JR-0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 -> (none)
- R201, R202: MPN (none) -> RT1206BRE07100RL; Supplier https://www.digikey.com/en/products/detail/yageo/RT1206BRE0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 -> (none)
- R203, R5: MPN (none) -> RC0402JR-07100RL; Supplier https://www.digikey.com/en/products/detail/yageo/RC0402JR-0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 -> (none)
- U201: MPN (none) -> TLV3603DCKR; Supplier https://www.digikey.com/en/products/detail/texas-instrument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 -> (none)
Changed lines of the file:
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@@
 			)
 		)
-		(property "Supplier" "https://www.digikey.com/en/products/detail/skyworks-solutions-inc/SMP1345-040LF/2217452"
+		(property "Supplier" ""
+			(at 25.4 66.04 90)
+			(effects
+				(font
+					(size 1.27 1.27)
+				)
+				(hide yes)
+			)
+		)
+		(property "MPN" "SMP1345-040LF"
 			(at 25.4 66.04 90)
 			(effects
@@
 			)
 		)
-		(property "Supplier" "https://www.digikey.com/en/products/detail/murata-electronics/GRM155R71C103KA01D/587215"
+		(property "Supplier" ""
+			(at 143.51 34.29 0)
+			(effects
+				(font
+					(size 1.27 1.27)
+				)
+				(hide yes)
+			)
+		)
+		(property "MPN" "GRM155R71C103KA01D"
 			(at 143.51 34.29 0)
 			(effects
@@
 			)
 		)
-		(property "Supplier" "https://www.digikey.com/en/products/detail/yageo/RC0402JR-07100RL/726415"
+		(property "Supplier" ""
+			(at 90.17 115.57 90)
+			(effects
+				(font
+					(size 1.27 1.27)
+				)
+				(hide yes)
+			)
+		)
+		(property "MPN" "RC0402JR-07100RL"
 			(at 90.17 115.57 90)
 			(effects
@@
 			)
 		)
-		(property "Supplier" "https://www.digikey.com/en/products/detail/skyworks-solutions-inc/SMP1345-040LF/2217452"
+		(property "Supplier" ""
+			(at 40.64 76.2 90)
+			(effects
+				(font
+					(size 1.27 1.27)
+				)
+				(hide yes)
+			)
+		)
+		(property "MPN" "SMP1345-040LF"
 			(at 40.64 76.2 90)
 			(effects
@@
 			)
 		)
-		(property "Supplier" "https://www.digikey.com/en/products/detail/yageo/RC0402JR-07100RL/726415"
+		(property "Supplier" ""
+			(at 53.34 132.08 90)
+			(effects
+				(font
+					(size 1.27 1.27)
+				)
+				(hide yes)
+			)
+		)
+		(property "MPN" "RC0402JR-071KL "
 			(at 53.34 132.08 90)
 			(effects
@@
 			)
 		)
-		(property "Supplier" "https://www.digikey.com/en/products/detail/skyworks-solutions-inc/SMP1345-040LF/2217452"
+		(property "Supplier" ""
+			(at 40.64 66.04 90)
+			(effects
+				(font
+					(size 1.27 1.27)
+				)
+				(hide yes)
+			)
+		)
+		(property "MPN" "SMP1345-040LF"
 			(at 40.64 66.04 90)
 			(effects
@@
 			)
 		)
-		(property "Supplier" "https://www.digikey.com/en/products/detail/skyworks-solutions-inc/SMP1345-040LF/2217452"
+		(property "Supplier" ""
+			(at 40.64 148.59 90)
+			(effects
+				(font
+					(size 1.27 1.27)
+				)
+				(hide yes)
+			)
+		)
+		(property "MPN" "SMP1345-040LF"
 			(at 40.64 148.59 90)
 			(effects
@@
 			)
 		)
-		(property "Supplier" "https://www.digikey.com/en/products/detail/yageo/CC0402JRNPO9BN101/302758"
+		(property "Supplier" ""
+			(at 128.27 34.29 0)
+			(effects
+				(font
+					(size 1.27 1.27)
+				)
+				(hide yes)
+			)
+		)
+		(property "MPN" "CC0402JRNPO9BN101"
 			(at 128.27 34.29 0)
 			(effects
@@
 			)
 		)
-		(property "Supplier" "https://www.digikey.com/en/products/detail/kyocera-avx/0402ZD105KAT2A/1545026"
+		(property "Supplier" ""
+			(at 158.75 34.29 0)
+			(effects
+				(font
+					(size 1.27 1.27)
+				)
+				(hide yes)
+			)
+		)
+		(property "MPN" "0402ZD105KAT2A"
 			(at 158.75 34.29 0)
 			(effects
@@
 			)
 		)
-		(property "Supplier" "https://www.digikey.com/en/products/detail/skyworks-solutions-inc/SMP1345-040LF/2217452"
+		(property "Supplier" ""
+			(at 25.4 148.59 90)
+			(effects
+				(font
+					(size 1.27 1.27)
+				)
+				(hide yes)
+			)
+		)
+		(property "MPN" "SMP1345-040LF"
 			(at 25.4 148.59 90)
 			(effects
@@
 			)
 		)
-		(property "Supplier" "https://www.digikey.com/en/products/detail/skyworks-solutions-inc/SMP1345-040LF/2217452"
+		(property "Supplier" ""
+			(at 25.4 76.2 90)
+			(effects
+				(font
+					(size 1.27 1.27)
+				)
+				(hide yes)
+			)
+		)
+		(property "MPN" "SMP1345-040LF"
 			(at 25.4 76.2 90)
 			(effects
@@
 			)
 		)
-		(property "Supplier" "https://www.digikey.com/en/products/detail/kyocera-avx/KGM05AR51C104KH/563236"
+		(property "Supplier" ""
+			(at 102.87 153.67 0)
+			(effects
+				(font
+					(size 1.27 1.27)
+				)
+				(hide yes)
+			)
+		)
+		(property "MPN" "KGM05AR51C104KH"
 			(at 102.87 153.67 0)
 			(effects
@@
 			)
 		)
-		(property "Supplier" "https://www.digikey.com/en/products/detail/yageo/RT1206BRE07100RL/1080028"
+		(property "Supplier" ""
+			(at 55.88 66.04 0)
+			(effects
+				(font
+					(size 1.27 1.27)
+				)
+				(hide yes)
+			)
+		)
+		(property "MPN" "RT1206BRE07100RL"
 			(at 55.88 66.04 0)
 			(effects
@@
 			)
 		)
-		(property "Supplier" "https://www.digikey.com/en/products/detail/skyworks-solutions-inc/SMP1345-040LF/2217452"
+		(property "Supplier" ""
+			(at 25.4 138.43 90)
+			(effects
+				(font
+					(size 1.27 1.27)
+				)
+				(hide yes)
+			)
+		)
+		(property "MPN" "SMP1345-040LF"
 			(at 25.4 138.43 90)
 			(effects
@@
 			)
 		)
-		(property "Supplier" "https://www.digikey.com/en/products/detail/yageo/RC0402JR-07100RL/726415"
+		(property "Supplier" ""
+			(at 88.9 59.69 90)
+			(effects
+				(font
+					(size 1.27 1.27)
+				)
+				(hide yes)
+			)
+		)
+		(property "MPN" "RC0402JR-07100RL"
 			(at 88.9 59.69 90)
 			(effects
@@
 			)
 		)
-		(property "Supplier" "https://www.digikey.com/en/products/detail/rohm-semiconductor/RBE01VYM6AFHTR/24634517?s=N4IgjCBcoKwOwAYqgMZQGYEMA2BnApgDQgBuAdlAC4BOArkSAPZQDaIALAggMxwAcIALrEADpSggAyjQCWZAOYgAvsTABOPmuQg0kLHgbNIbJIJUgATBYBsEaDow4CxI2wtcABAFsAah4ACHnAAdDDeAIJCouKQIADCjLQi2PgAJgCqZDKUAPLoALL4mLi01PjKxAC0Wva6NPQurOBC5pUW2nV0hk0wLebW2jKpEpVgCBDREiDElACeIuWxxWhKSkA"
+		(property "Supplier" ""
+			(at 59.69 138.43 90)
+			(effects
+				(font
+					(size 1.27 1.27)
+				)
+				(hide yes)
+			)
+		)
+		(property "MPN" "RBE01VYM6AFHTR"
 			(at 59.69 138.43 90)
 			(effects
@@
 			)
 		)
-		(property "Supplier" "https://www.digikey.com/en/products/detail/yageo/RT1206BRE07100RL/1080028"
+		(property "Supplier" ""
+			(at 68.58 66.04 0)
+			(effects
+				(font
+					(size 1.27 1.27)
+				)
+				(hide yes)
+			)
+		)
+		(property "MPN" "RT1206BRE07100RL"
 			(at 68.58 66.04 0)
 			(effects
@@
 			)
 		)
-		(property "Supplier" "https://www.digikey.com/en/products/detail/skyworks-solutions-inc/SMP1345-040LF/2217452"
+		(property "Supplier" ""
+			(at 40.64 138.43 90)
+			(effects
+				(font
+					(size 1.27 1.27)
+				)
+				(hide yes)
+			)
+		)
+		(property "MPN" "SMP1345-040LF"
 			(at 40.64 138.43 90)
 			(effects
@@
 			)
 		)
-		(property "Supplier" "https://www.digikey.com/en/products/detail/texas-instruments/TLV3603DCKR/15853830"
+		(property "Supplier" ""
 			(at 102.87 62.23 0)
 			(effects
+				(font
+					(size 1.27 1.27)
+				)
+				(hide yes)
+			)
+		)
+		(property "MPN" "TLV3603DCKR"
+			(at 102.87 62.23 0)
+			(effects

Commit message: finish 2.0 part selection
Parts:
- C1: footprint (none) -> Custom:C_0402_1005Metric_Fix; MPN (none) -> GRM1555C1H332JE01D
- C2: footprint (none) -> Custom:C_0402_1005Metric_Fix; MPN (none) -> CC0402JRNPO9BN101
- C3: footprint (none) -> Custom:C_0402_1005Metric_Fix; MPN (none) -> KGM05AR51C104KH
- R1: footprint (none) -> Custom:R_0402_1005Metric_Fix; MPN (none) -> RC0402JR-13330RL
- RFC1: footprint (none) -> Inductor_SMD:L_0603_1608Metric; MPN (none) -> 7447610260
- RFC2: footprint (none) -> Inductor_SMD:L_0805_2012Metric; MPN (none) -> BRC2012T3R3MD
- U1: MPN (none) -> NCS2250SN2T1G
Changed lines of the file:
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@@
 	(title_block
 		(title "Frequency Counter")
-		(date "2026-02-17")
+		(date "2026-02-18")
 		(rev "2.0-draft")
 		(company "vladaviedov.org")
@@
 			)
 		)
-		(property "Supplier" ""
-			(at 25.4 66.04 90)
-			(effects
-				(font
-					(size 1.27 1.27)
-				)
-				(hide yes)
-			)
-		)
 		(property "MPN" "SMP1345-040LF"
 			(at 25.4 66.04 90)
@@
 			)
 		)
+		(property "MPN" "NCS2250SN2T1G"
+			(at 91.44 134.62 0)
+			(effects
+				(font
+					(size 1.27 1.27)
+				)
+				(hide yes)
+			)
+		)
 		(pin "2"
 		)
@@
 			)
 		)
-		(property "Supplier" ""
-			(at 143.51 34.29 0)
-			(effects
-				(font
-					(size 1.27 1.27)
-				)
-				(hide yes)
-			)
-		)
 		(property "MPN" "GRM155R71C103KA01D"
 			(at 143.51 34.29 0)
@@
 			)
 		)
-		(property "Supplier" ""
-			(at 90.17 115.57 90)
-			(effects
-				(font
-					(size 1.27 1.27)
-				)
-				(hide yes)
-			)
-		)
 		(property "MPN" "RC0402JR-07100RL"
 			(at 90.17 115.57 90)
@@
 			)
 		)
-		(property "Supplier" ""
-			(at 40.64 76.2 90)
-			(effects
-				(font
-					(size 1.27 1.27)
-				)
-				(hide yes)
-			)
-		)
 		(property "MPN" "SMP1345-040LF"
 			(at 40.64 76.2 90)
@@
 			)
 		)
-		(property "Supplier" ""
-			(at 53.34 132.08 90)
-			(effects
-				(font
-					(size 1.27 1.27)
-				)
-				(hide yes)
-			)
-		)
 		(property "MPN" "RC0402JR-071KL "
 			(at 53.34 132.08 90)
@@
 			)
 		)
-		(property "Footprint" ""
+		(property "Footprint" "Custom:C_0402_1005Metric_Fix"
 			(at 78.74 58.7248 0)
 			(effects
@@
 			)
 		)
+		(property "MPN" "GRM1555C1H332JE01D"
+			(at 74.93 59.69 90)
+			(effects
+				(font
+					(size 1.27 1.27)
+				)
+				(hide yes)
+			)
+		)
 		(pin "2"
 		)
@@
 			)
 		)
-		(property "Footprint" ""
+		(property "Footprint" "Custom:C_0402_1005Metric_Fix"
 			(at 91.44 39.6748 0)
 			(effects
@@
 			)
 		)
+		(property "MPN" "CC0402JRNPO9BN101"
+			(at 87.63 40.64 90)
+			(effects
+				(font
+					(size 1.27 1.27)
+				)
+				(hide yes)
+			)
+		)
 		(pin "2"
 		)
@@
 			)
 		)
-		(property "Supplier" ""
-			(at 40.64 66.04 90)
-			(effects
-				(font
-					(size 1.27 1.27)
-				)
-				(hide yes)
-			)
-		)
 		(property "MPN" "SMP1345-040LF"
 			(at 40.64 66.04 90)
@@
 			)
 		)
-		(property "Footprint" ""
+		(property "Footprint" "Custom:R_0402_1005Metric_Fix"
 			(at 98.044 39.624 90)
 			(effects
@@
 			)
 		)
+		(property "MPN" "RC0402JR-13330RL"
+			(at 97.79 40.64 90)
+			(effects
+				(font
+					(size 1.27 1.27)
+				)
+				(hide yes)
+			)
+		)
 		(pin "1"
 		)
@@
 			)
 		)
-		(property "Supplier" ""
-			(at 40.64 148.59 90)
-			(effects
-				(font
-					(size 1.27 1.27)
-				)
-				(hide yes)
-			)
-		)
 		(property "MPN" "SMP1345-040LF"
 			(at 40.64 148.59 90)
@@
 			)
 		)
-		(property "Supplier" ""
-			(at 128.27 34.29 0)
-			(effects
-				(font
-					(size 1.27 1.27)
-				)
-				(hide yes)
-			)
-		)
 		(property "MPN" "CC0402JRNPO9BN101"
 			(at 128.27 34.29 0)
@@
 			)
 		)
-		(property "Supplier" ""
-			(at 158.75 34.29 0)
-			(effects
-				(font
-					(size 1.27 1.27)
-				)
-				(hide yes)
-			)
-		)
 		(property "MPN" "0402ZD105KAT2A"
 			(at 158.75 34.29 0)
@@
 			)
 		)
-		(property "Supplier" ""
-			(at 25.4 148.59 90)
-			(effects
-				(font
-					(size 1.27 1.27)
-				)
-				(hide yes)
-			)
-		)
 		(property "MPN" "SMP1345-040LF"
 			(at 25.4 148.59 90)
@@
 			)
 		)
-		(property "Supplier" ""
-			(at 25.4 76.2 90)
-			(effects
-				(font
-					(size 1.27 1.27)
-				)
-				(hide yes)
-			)
-		)
 		(property "MPN" "SMP1345-040LF"
 			(at 25.4 76.2 90)
@@
 			)
 		)
-		(property "Supplier" ""
-			(at 102.87 153.67 0)
-			(effects
-				(font
-					(size 1.27 1.27)
-				)
-				(hide yes)
-			)
-		)
 		(property "MPN" "KGM05AR51C104KH"
 			(at 102.87 153.67 0)
@@
 			)
 		)
-		(property "Supplier" ""
-			(at 55.88 66.04 0)
-			(effects
-				(font
-					(size 1.27 1.27)
-				)
-				(hide yes)
-			)
-		)
 		(property "MPN" "RT1206BRE07100RL"
 			(at 55.88 66.04 0)
@@
 			)
 		)
-		(property "Footprint" ""
+		(property "Footprint" "Custom:C_0402_1005Metric_Fix"
 			(at 91.44 26.9748 0)
 			(effects
@@
 			)
 		)
+		(property "MPN" "KGM05AR51C104KH"
+			(at 87.63 27.94 90)
+			(effects
+				(font
+					(size 1.27 1.27)
+				)
+				(hide yes)
+			)
+		)
 		(pin "2"
 		)
@@
 			)
 		)
-		(property "Supplier" ""
-			(at 25.4 138.43 90)
-			(effects
-				(font
-					(size 1.27 1.27)
-				)
-				(hide yes)
-			)
-		)
 		(property "MPN" "SMP1345-040LF"
 			(at 25.4 138.43 90)
@@
 			)
 		)
-		(property "Footprint" ""
+		(property "Footprint" "Inductor_SMD:L_0805_2012Metric"
 			(at 81.28 34.29 0)
 			(effects
@@
 			)
 		)
+		(property "MPN" "BRC2012T3R3MD"
+			(at 81.28 34.29 0)
+			(effects
+				(font
+					(size 1.27 1.27)
+				)
+				(hide yes)
+			)
+		)
 		(pin "2"
 		)
@@
 			)
 		)
-		(property "Supplier" ""
-			(at 88.9 59.69 90)
-			(effects
-				(font
-					(size 1.27 1.27)
-				)
-				(hide yes)
-			)
-		)
 		(property "MPN" "RC0402JR-07100RL"
 			(at 88.9 59.69 90)
@@
 			)
 		)
-		(property "Supplier" ""
-			(at 59.69 138.43 90)
-			(effects
-				(font
-					(size 1.27 1.27)
-				)
-				(hide yes)
-			)
-		)
 		(property "MPN" "RBE01VYM6AFHTR"
 			(at 59.69 138.43 90)
@@
 			)
 		)
-		(property "Supplier" ""
-			(at 68.58 66.04 0)
-			(effects
-				(font
-					(size 1.27 1.27)
-				)
-				(hide yes)
-			)
-		)
 		(property "MPN" "RT1206BRE07100RL"
 			(at 68.58 66.04 0)
@@
 			)
 		)
-		(property "Supplier" ""
-			(at 40.64 138.43 90)
-			(effects
-				(font
-					(size 1.27 1.27)
-				)
-				(hide yes)
-			)
-		)
 		(property "MPN" "SMP1345-040LF"
 			(at 40.64 138.43 90)
@@
 			)
 		)
-		(property "Supplier" ""
-			(at 102.87 62.23 0)
-			(effects
-				(font
-					(size 1.27 1.27)
-				)
-				(hide yes)
-			)
-		)
 		(property "MPN" "TLV3603DCKR"
 			(at 102.87 62.23 0)
@@
 			)
 		)
-		(property "Footprint" ""
+		(property "Footprint" "Inductor_SMD:L_0603_1608Metric"
 			(at 81.28 46.99 0)
 			(effects
@@
 			(at 81.28 46.99 0)
 			(effects
+				(font
+					(size 1.27 1.27)
+				)
+				(hide yes)
+			)
+		)
+		(property "MPN" "7447610260"
+			(at 81.28 46.99 0)
+			(effects

Commit message: assign references
Parts:
- renumbered C1 to C201, C3 to C202, C2 to C203, CD1 to CD204, D1 to D202, D202 to D203, D2 to D204, D3 to D205, D4 to D206, D5 to D207, D6 to D208, D203 to D209, RFC2 to L201, RFC1 to L202, R1 to R204, R2 to R205, R5 to R206, U1 to U202
