File: kicad/reference_clock.kicad_sch (KiCad schematic)
At the start: 11 parts, among them U301 74AHC1G4210, U302 74VHC4040FT, U303 74HC251PW, Y301 32.768kHz

Commit message: redesign pierce oscillator
Parts:
- C301: value 33pF -> 22pF
- C302: value 100pF -> 22pF
- R301: value 100k -> 1Meg; footprint Custom:R_0402_1005Metric_Fix -> (none); Supplier https://www.digikey.com/en/products/detail/yageo/RC0402JR-0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 -> (none)
- R302: footprint Custom:R_0402_1005Metric_Fix -> (none)
- renumbered CD303 to CD301, CD301 to CD302, CD302 to CD303, U303 to U302, U302 to U303
Connections:
- net at R301.1, U301.1 (X1), Y301.2: now also C301.1
- net at R301.2, U301.2 (X2): now also R302.1; no longer R302.2
- net at C302.1, Y301.1: now also R302.2; no longer C301.1, R302.1
Other:
- moved on the sheet: C301, C302, CD302, CD303, U301, U303, Y301

Commit message: replace alum caps with ceramics, change mpn labeling
Parts:
- CD301, CD302, CD303: MPN (none) -> KGM05AR51C104KH; Supplier https://www.digikey.com/en/products/detail/kyocera-avx/KGM0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 -> (none)
- R302: MPN (none) -> RC0402JR-132K2L; Supplier https://www.digikey.com/en/products/detail/yageo/RC0402JR-1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 -> (none)
- U301: MPN (none) -> 74AHC1G4210GWH; Supplier https://www.digikey.com/en/products/detail/nexperia-usa-inc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 -> (none)
- U302: MPN (none) -> 74HC251PW,118; Supplier https://www.digikey.com/en/products/detail/nexperia-usa-inc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 -> (none)
- U303: MPN (none) -> 74VHC4040FT; Supplier https://www.digikey.com/en/products/detail/toshiba-semicond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 -> (none)
Changed lines of the file:
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@@
 			)
 		)
-		(property "Supplier" "https://www.digikey.com/en/products/detail/kyocera-avx/KGM05AR51C104KH/563236"
+		(property "Supplier" ""
+			(at 21.59 123.19 0)
+			(effects
+				(font
+					(size 1.27 1.27)
+				)
+				(hide yes)
+			)
+		)
+		(property "MPN" "KGM05AR51C104KH"
 			(at 21.59 123.19 0)
 			(effects
@@
 			)
 		)
-		(property "Supplier" "https://www.digikey.com/en/products/detail/nexperia-usa-inc/74AHC1G4210GWH/7495486"
+		(property "Supplier" ""
+			(at 49.53 40.64 0)
+			(effects
+				(font
+					(size 1.27 1.27)
+				)
+				(hide yes)
+			)
+		)
+		(property "MPN" "74AHC1G4210GWH"
 			(at 49.53 40.64 0)
 			(effects
@@
 			)
 		)
-		(property "Supplier" "https://www.digikey.com/en/products/detail/yageo/RC0402JR-132K2L/13694130"
+		(property "Supplier" ""
+			(at 36.83 55.88 0)
+			(effects
+				(font
+					(size 1.27 1.27)
+				)
+				(hide yes)
+			)
+		)
+		(property "MPN" "RC0402JR-132K2L"
 			(at 36.83 55.88 0)
 			(effects
@@
 			)
 		)
-		(property "Supplier" "https://www.digikey.com/en/products/detail/kyocera-avx/KGM05AR51C104KH/563236"
+		(property "Supplier" ""
+			(at 97.79 62.23 0)
+			(effects
+				(font
+					(size 1.27 1.27)
+				)
+				(hide yes)
+			)
+		)
+		(property "MPN" "KGM05AR51C104KH"
 			(at 97.79 62.23 0)
 			(effects
@@
 			)
 		)
-		(property "Supplier" "https://www.digikey.com/en/products/detail/nexperia-usa-inc/74HC251PW-118/1230237"
+		(property "Supplier" ""
+			(at 69.85 128.27 0)
+			(effects
+				(font
+					(size 1.27 1.27)
+				)
+				(hide yes)
+			)
+		)
+		(property "MPN" "74HC251PW,118"
 			(at 69.85 128.27 0)
 			(effects
@@
 			)
 		)
-		(property "Supplier" "https://www.digikey.com/en/products/detail/toshiba-semiconductor-and-storage/74VHC4040FT/5155784"
+		(property "Supplier" ""
+			(at 120.65 50.8 0)
+			(effects
+				(font
+					(size 1.27 1.27)
+				)
+				(hide yes)
+			)
+		)
+		(property "MPN" "74VHC4040FT"
 			(at 120.65 50.8 0)
 			(effects
@@
 			)
 		)
-		(property "Supplier" "https://www.digikey.com/en/products/detail/kyocera-avx/KGM05AR51C104KH/563236"
+		(property "Supplier" ""
 			(at 64.77 64.77 0)
 			(effects
+				(font
+					(size 1.27 1.27)
+				)
+				(hide yes)
+			)
+		)
+		(property "MPN" "KGM05AR51C104KH"
+			(at 64.77 64.77 0)
+			(effects

Commit message: finish 2.0 part selection
Parts:
- C301, C302: MPN (none) -> GRM1555C1H220JA01D; Supplier https://www.digikey.com/en/products/detail/murata-electroni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 -> (none)
- R301: footprint (none) -> Custom:R_0402_1005Metric_Fix; MPN (none) -> RC0402FR-071ML
- R302: footprint (none) -> Custom:R_0402_1005Metric_Fix
- Y301: footprint Crystal:Crystal_SMD_G8-2Pin_3.2x1.5mm -> Crystal:Crystal_SMD_EuroQuartz_EQ161-2Pin_3.2x1.5mm_HandSoldering; MPN (none) -> CM315D32768HZFT; Supplier https://www.digikey.com/en/products/detail/abracon-llc/ABS0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 -> (none)
Changed lines of the file:
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@@
 	(title_block
 		(title "Frequency Counter")
-		(date "2026-02-17")
+		(date "2026-02-18")
 		(rev "2.0-draft")
 		(company "vladaviedov.org")
@@
 			)
 		)
-		(property "Footprint" ""
+		(property "Footprint" "Custom:R_0402_1005Metric_Fix"
 			(at 29.464 47.244 90)
 			(effects
@@
 		(property "Description" "Resistor, US symbol"
 			(at 29.21 48.26 0)
+			(effects
+				(font
+					(size 1.27 1.27)
+				)
+				(hide yes)
+			)
+		)
+		(property "MPN" "RC0402FR-071ML"
+			(at 29.21 48.26 90)
 			(effects
 				(font
@@
 			)
 		)
-		(property "Supplier" ""
-			(at 21.59 123.19 0)
-			(effects
-				(font
-					(size 1.27 1.27)
-				)
-				(hide yes)
-			)
-		)
 		(property "MPN" "KGM05AR51C104KH"
 			(at 21.59 123.19 0)
@@
 		)
 		(property "Description" "10-stage divider and oscillator, SOT353-1"
-			(at 49.53 40.64 0)
-			(effects
-				(font
-					(size 1.27 1.27)
-				)
-				(hide yes)
-			)
-		)
-		(property "Supplier" ""
 			(at 49.53 40.64 0)
 			(effects
@@
 			)
 		)
-		(property "Footprint" ""
+		(property "Footprint" "Custom:R_0402_1005Metric_Fix"
 			(at 37.846 56.134 90)
 			(effects
@@
 		)
 		(property "Description" "Resistor, US symbol"
-			(at 36.83 55.88 0)
-			(effects
-				(font
-					(size 1.27 1.27)
-				)
-				(hide yes)
-			)
-		)
-		(property "Supplier" ""
 			(at 36.83 55.88 0)
 			(effects
@@
 			)
 		)
-		(property "Supplier" ""
-			(at 97.79 62.23 0)
-			(effects
-				(font
-					(size 1.27 1.27)
-				)
-				(hide yes)
-			)
-		)
 		(property "MPN" "KGM05AR51C104KH"
 			(at 97.79 62.23 0)
@@
 			)
 		)
-		(property "Supplier" ""
-			(at 69.85 128.27 0)
-			(effects
-				(font
-					(size 1.27 1.27)
-				)
-				(hide yes)
-			)
-		)
 		(property "MPN" "74HC251PW,118"
 			(at 69.85 128.27 0)
@@
 			)
 		)
-		(property "Supplier" ""
-			(at 120.65 50.8 0)
-			(effects
-				(font
-					(size 1.27 1.27)
-				)
-				(hide yes)
-			)
-		)
 		(property "MPN" "74VHC4040FT"
 			(at 120.65 50.8 0)
@@
 			)
 		)
-		(property "Footprint" "Crystal:Crystal_SMD_G8-2Pin_3.2x1.5mm"
+		(property "Footprint" "Crystal:Crystal_SMD_EuroQuartz_EQ161-2Pin_3.2x1.5mm_HandSoldering"
 			(at 29.21 63.5 0)
 			(effects
@@
 			)
 		)
-		(property "Supplier" "https://www.digikey.com/en/products/detail/abracon-llc/ABS07-32-768KHZ-T/1236858"
-			(at 29.21 63.5 90)
+		(property "MPN" "CM315D32768HZFT"
+			(at 29.21 63.5 0)
 			(effects
 				(font
@@
 			)
 		)
-		(property "Supplier" ""
-			(at 64.77 64.77 0)
-			(effects
-				(font
-					(size 1.27 1.27)
-				)
-				(hide yes)
-			)
-		)
 		(property "MPN" "KGM05AR51C104KH"
 			(at 64.77 64.77 0)
@@
 			)
 		)
-		(property "Supplier" "https://www.digikey.com/en/products/detail/murata-electronics/GRM1555C1H101GA01D/3693920"
+		(property "MPN" "GRM1555C1H220JA01D"
 			(at 36.83 71.12 0)
 			(effects
@@
 			)
 		)
-		(property "Supplier" "https://www.digikey.com/en/products/detail/murata-electronics/GRM1555C1H330GA01J/4358133"
+		(property "MPN" "GRM1555C1H220JA01D"
 			(at 21.59 71.12 0)
 			(effects

Commit message: assign references
Parts:
- renumbered CD302 to CD301, CD303 to CD302, CD301 to CD303, U303 to U302, U302 to U303
Changed lines of the file:
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@@
 		(dnp no)
 		(fields_autoplaced yes)
-		(property "Reference" "CD301"
+		(property "Reference" "CD303"
 			(at 25.4 121.9199 0)
 			(effects
@@
 			(project "frequency_counter"
 				(path "/62339e8b-4e00-440f-8d81-4472a4f50c26/ad3ea9b5-9e07-4330-8c93-7bb022b6949a"
-					(reference "CD301")
+					(reference "CD303")
 					(unit 1)
 				)
@@
 		(dnp no)
 		(fields_autoplaced yes)
-		(property "Reference" "CD303"
+		(property "Reference" "CD302"
 			(at 101.6 60.9599 0)
 			(effects
@@
 			(project "frequency_counter"
 				(path "/62339e8b-4e00-440f-8d81-4472a4f50c26/ad3ea9b5-9e07-4330-8c93-7bb022b6949a"
-					(reference "CD303")
+					(reference "CD302")
 					(unit 1)
 				)
@@
 		(dnp no)
 		(fields_autoplaced yes)
-		(property "Reference" "U302"
+		(property "Reference" "U303"
 			(at 71.9933 105.41 0)
 			(effects
@@
 			(project ""
 				(path "/62339e8b-4e00-440f-8d81-4472a4f50c26/ad3ea9b5-9e07-4330-8c93-7bb022b6949a"
-					(reference "U302")
+					(reference "U303")
 					(unit 1)
 				)
@@
 		(dnp no)
 		(fields_autoplaced yes)
-		(property "Reference" "U303"
+		(property "Reference" "U302"
 			(at 122.7933 30.48 0)
 			(effects
@@
 			(project "frequency_counter"
 				(path "/62339e8b-4e00-440f-8d81-4472a4f50c26/ad3ea9b5-9e07-4330-8c93-7bb022b6949a"
-					(reference "U303")
+					(reference "U302")
 					(unit 1)
 				)
@@
 		(dnp no)
 		(fields_autoplaced yes)
-		(property "Reference" "CD302"
+		(property "Reference" "CD301"
 			(at 68.58 63.4999 0)
 			(effects
@@
 			(project "frequency_counter"
 				(path "/62339e8b-4e00-440f-8d81-4472a4f50c26/ad3ea9b5-9e07-4330-8c93-7bb022b6949a"
-					(reference "CD302")
-					(unit 1)
-				)
+					(reference "CD301")
+					(unit 1)
+				)

Commit message: minor fixes, 2.0 schematic
Connections:
- net +5V: no longer U303.7 (~{OE})
- net GND: now also U303.7 (~{OE})
