File: kicad/frequency_counter.kicad_pcb (KiCad board)
At the start: 4 copper layers, 75 x 100 mm, 104 parts, among them J101 CH.A, J102 J, J103 DISPLAY, J601 AVR-ISP-6, Q701 SIL2300, SW101 SPDT, SW102 PEC12R, U201 TLV3603DCK, U301 74AHC1G4210, U302 74VHC4040FT, U303 74HC251PW, U401 74LVC1G02W5, U402 74LVC1G80GW, U403 74HC04PW, U404 74LVC1G80GW, U405 74VHC4040FT, U406 74VHC4040FT, U407 74VHC4040FT, U501 74HC165D, U502 74HC165D, U503 74HC165D, U504 74HC165D, U601 ATtiny1634-S, U701 TP4057, U702 DW01, U703 TPS613222ADBV, Y301 32.768kHz

Commit message: redesign pcb for 2.0
Parts:
- removed C701, C702: 4.7uF, Capacitor_THT:CP_Radial_D5.0mm_P2.00mm
- removed C705: 22uF, Capacitor_THT:CP_Radial_D5.0mm_P2.00mm
- removed JP601: NORMAL/~{PROG}, Custom:TestPoint_2Pads_Pitch2.54mm_Drill0.8mm_Fix
- removed REF**: Symbol_Attention_Triangle_6mm_Silkscreen, Custom:Symbol_Attention_Triangle_6mm_Silkscreen
- removed REF**: KiCad-Logo2_5mm_SilkScreen, Symbol:KiCad-Logo2_5mm_SilkScreen
- removed TP401: TestPoint, Custom:TestPoint_Pad_2.0x2.0mm_Fix
- added C201: 3.3nF, Custom:C_0402_1005Metric_Fix, F.Cu at (108.9, 71.1)
- added C202: 0.1uF, Custom:C_0402_1005Metric_Fix, F.Cu at (101.4, 75.0)
- added C203: 100pF, Custom:C_0402_1005Metric_Fix, F.Cu at (104.8, 71.1)
- added C801: 10uF, Capacitor_SMD:C_0603_1608Metric, F.Cu at (158.2, 137.8)
- added C802: 10uF, Capacitor_SMD:C_0603_1608Metric, F.Cu at (151.9, 138.1)
- added C805: 10uF, Capacitor_SMD:C_0603_1608Metric, F.Cu at (157.4, 116.7)
- added CD204: 0.1uF, Custom:C_0402_1005Metric_Fix, F.Cu at (142.5, 61.4)
- added CD407: 100pF, Custom:C_0402_1005Metric_Fix, F.Cu at (117.2, 71.1)
- added CD408: 0.1uF, Custom:C_0402_1005Metric_Fix, F.Cu at (116.2, 71.1)
- added CD409: 0.1uF, Custom:C_0402_1005Metric_Fix, F.Cu at (123.5, 75.3)
- added CD411: 0.1uF, Custom:C_0402_1005Metric_Fix, F.Cu at (124.9, 73.4)
- added CD802: 0.1uF, Custom:C_0402_1005Metric_Fix, F.Cu at (101.0, 77.4)
- added D204: SMP1345, Diode_SMD:D_0402_1005Metric_Pad0.77x0.64mm_HandSolder, F.Cu at (112.9, 67.3)
- added D205: SMP1345, Diode_SMD:D_0402_1005Metric_Pad0.77x0.64mm_HandSolder, F.Cu at (135.9, 61.9)
- added D206: SMP1345, Diode_SMD:D_0402_1005Metric_Pad0.77x0.64mm_HandSolder, F.Cu at (134.9, 61.9)
- added D207: SMP1345, Diode_SMD:D_0402_1005Metric_Pad0.77x0.64mm_HandSolder, F.Cu at (135.9, 64.4)
- added D208: SMP1345, Diode_SMD:D_0402_1005Metric_Pad0.77x0.64mm_HandSolder, F.Cu at (134.9, 64.4)
- added D209: RBE01VYM6AFH, Diode_SMD:D_SOD-323_HandSoldering, F.Cu at (138.5, 64.6)
- added J102: SMA, Custom:SMA_Adjusted, F.Cu at (126.1, 62.1)
- added L201: 3.3uH, Inductor_SMD:L_0805_2012Metric, F.Cu at (101.5, 72.7)
- added L202: 600nH, Inductor_SMD:L_0603_1608Metric, F.Cu at (106.9, 72.0)
- added R101: 4.7k, Custom:R_0402_1005Metric_Fix, F.Cu at (132.2, 96.0)
- added R102: 4.7k, Custom:R_0402_1005Metric_Fix, F.Cu at (129.7, 96.0)
- added R204: 330, Custom:R_0402_1005Metric_Fix, F.Cu at (106.3, 70.7)
- added R205: 1k, Custom:R_0402_1005Metric_Fix, F.Cu at (137.4, 63.1)
- added R206: 100k, Custom:R_0402_1005Metric_Fix, F.Cu at (137.9, 61.6)
- added R808: 10k, Custom:R_0402_1005Metric_Fix, F.Cu at (99.8, 81.4)
- added SW101: PushBtn, Button_Switch_SMD:SW_Push_1P1T_NO_E-Switch_TL3301NxxxxxG, F.Cu at (123.7, 132.9)
- added U202: NCS2250, Package_SO:TSOP-5_1.65x3.05mm_P0.95mm, F.Cu at (140.2, 61.8)
- added U405: 74LVC1G80GW, Package_TO_SOT_SMD:SOT-353_SC-70-5, F.Cu at (116.5, 73.4)
- added U406: 7UL2G00FK, Package_SO:VSSOP-8_2.3x2mm_P0.5mm, F.Cu at (121.7, 74.8)
- added U407: 74LVC1G157, Package_SO:TSOP-6_1.65x3.05mm_P0.95mm, F.Cu at (124.4, 70.6)
- added U804: LM4040D25FTA, Package_TO_SOT_SMD:SOT-23-3, F.Cu at (99.7, 83.7)
- added U805: MCP6001, Package_TO_SOT_SMD:SOT-353_SC-70-5, F.Cu at (99.6, 79.5)
- BT101: footprint Connector_Wire:SolderWire-0.5sqmm_1x02_P4.6mm_D0.9mm_OD2.1mm -> Connector_JST:JST_ZH_B2B-ZR_1x02_P1.50mm_Vertical
- C301: renamed from C302; value 100pF -> 22pF
- C302: renamed from C301; value 33pF -> 22pF
- C804: renamed from C704; value 1uF -> 10uF; footprint Custom:C_0402_1005Metric_Fix -> Capacitor_SMD:C_0603_1608Metric
- CD401: value 100pF -> 0.1uF
- CD410: value 0.1uF -> 100pF
- D203: value RBE01VYM6AFH -> SMP1345; footprint Diode_SMD:D_SOD-323_HandSoldering -> Diode_SMD:D_0402_1005Metric_Pad0.77x0.64mm_HandSolder
- J101: value CH.A -> SMA
- J104: renamed from J102; value J -> USB-C
- R203: value 470 -> 100
- R301: value 100k -> 1Meg
- SW102: value PEC12R -> PushBtn; footprint Rotary_Encoder:RotaryEncoder_Alps_EC11E-Switch_Vertical_H20mm -> Button_Switch_SMD:SW_Push_1P1T_NO_E-Switch_TL3301NxxxxxG
- SW103: renamed from SW101; value SPDT -> Rocker; footprint Connector_Wire:SolderWire-0.5sqmm_1x03_P4.6mm_D0.9mm_OD2.1mm -> Connector_Wire:SolderWire-1.5sqmm_1x02_P6mm_D1.7mm_OD3mm
- TP101: renamed from TP102; value TestPoint -> RCW; footprint Custom:TestPoint_Pad_2.0x2.0mm_Fix -> Custom:TestPoint_KOA_RCW
- TP102: renamed from TP101; value TestPoint -> RCW; footprint Custom:TestPoint_Pad_2.0x2.0mm_Fix -> Custom:TestPoint_KOA_RCW
- U401: value 74LVC1G02W5 -> 7UL2G00FK; footprint Package_TO_SOT_SMD:SC-74A-5_1.55x2.9mm_P0.95mm -> Package_SO:VSSOP-8_2.3x2mm_P0.5mm
- U402: value 74LVC1G80GW -> 7UL2G00FK; footprint Package_TO_SOT_SMD:SOT-353_SC-70-5 -> Package_SO:VSSOP-8_2.3x2mm_P0.5mm
- U403: value 74HC04PW -> 74LVC1G02W5; footprint Package_SO:TSSOP-14_4.4x5mm_P0.65mm -> Package_TO_SOT_SMD:SC-74A-5_1.55x2.9mm_P0.95mm
- Y301: footprint Crystal:Crystal_SMD_G8-2Pin_3.2x1.5mm -> Crystal:Crystal_SMD_EuroQuartz_EQ161-2Pin_3.2x1.5mm_HandSoldering
- moved CD402 20.4 mm to (133.2, 66.1), turned to 0 degrees
- moved U402 16.3 mm to (129.9, 66.8)
- moved CD401 15.1 mm to (104.7, 86.2), turned to 180 degrees
- moved SW102 13.9 mm to (136.9, 132.8)
- moved U403 11.1 mm to (112.4, 76.9), turned to 0 degrees
- moved U401 9.59 mm to (107.4, 84.4), turned to 180 degrees
- moved CD410 7.95 mm to (123.9, 73.4)
- moved D203 6.73 mm to (110.3, 67.3)
- moved U404 6.30 mm to (116.5, 77.8), turned to 0 degrees
- moved D202 6.25 mm to (105.3, 67.3), turned to 0 degrees
- moved TP101 6.07 mm to (106.9, 92.1)
- moved CD404 5.75 mm to (112.1, 74.2)
- moved CD406 5.68 mm to (116.9, 75.6), turned to 90 degrees
- moved CD201 5.66 mm to (105.5, 74.3), turned to 180 degrees
- moved CD202 5.59 mm to (105.5, 76.3), turned to 180 degrees
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- renumbered C703 to C803, CD407 to CD501, CD408 to CD502, CD409 to CD503, CD501 to CD601, CD502 to CD602, CD503 to CD603, CD504 to CD604, CD601 to CD701, CD701 to CD801, D601 to D701, D701 to D801, D702 to D802, D703 to D803, D704 to D804, J601 to J701, L701 to L801, Q701 to Q801, R101 to R105, R102 to R106, R603 to R701, R602 to R702, R601 to R703, R604 to R704, R605 to R705, R701 to R801, R702 to R802, R703 to R803, R704 to R804, R705 to R805, R706 to R806, R707 to R807, U405 to U501, U406 to U502, U407 to U503, U501 to U601, U502 to U602, U503 to U603, U504 to U604, U601 to U701, U701 to U801, U702 to U802, U703 to U803
Connections:
- C301 pad 1: Net-(C301-Pad1) -> Net-(U301-X1)
- C302 pad 1: Net-(C301-Pad1) -> Net-(C302-Pad1)
- CD701 pad 1: /Microcontroller/ISP.VCC -> +5V
- D201 pad 1: GND -> Net-(D201-K)
- D201 pad 2: /Frontend/RF -> /Frontend/CH_A
- D202 pad 1: /Frontend/RF -> GND
- D202 pad 2: GND -> Net-(D201-K)
- D203 pad 1: Net-(D203-K) -> /Frontend/CH_A
- D203 pad 2: GND -> Net-(D203-A)
- D701 pad 1: GND -> Net-(D701-K)
- D701 pad 2: Net-(D601-A) -> +5V
- J101 pad 1: /Frontend/RF -> /Frontend/CH_A
- J103 pad 3: /Microcontroller/ISP.SCK -> /Microcontroller/DISP_SCL
- J103 pad 4: /Microcontroller/ISP.MOSI -> /Microcontroller/DISP_SDA
- J701 pad 1: Net-(J601-MISO) -> /Microcontroller/ISP.MISO
- J701 pad 2: /Microcontroller/ISP.VCC -> +5V
- J701 pad 3: Net-(J601-SCK) -> /Microcontroller/ISP.SCK
- J701 pad 4: Net-(J601-MOSI) -> /Microcontroller/ISP.MOSI
- J701 pad 5: /Microcontroller/REF_DIV0 -> /Microcontroller/ISP.RST
- R201 pad 2: /Frontend/RF -> /Frontend/CH_A
- R202 pad 2: /Frontend/RF -> /Frontend/CH_A
- R203 pad 1: /Frontend/RF -> Net-(C201-Pad2)
- R203 pad 2: Net-(D203-K) -> Net-(U201-+)
- R302 pad 1: Net-(C301-Pad1) -> Net-(U301-X2)
- R302 pad 2: Net-(U301-X2) -> Net-(C302-Pad1)
- R701 pad 2: Net-(J601-SCK) -> Net-(U701-PC1)
- R702 pad 1: /Microcontroller/ISP.MOSI -> /Microcontroller/REF_RESET
- R702 pad 2: Net-(J601-MOSI) -> /Microcontroller/ISP.MOSI
- R703 pad 2: Net-(J601-MISO) -> /Measurement Unit/RESET
- R704 pad 1: /Microcontroller/ISP.VCC -> +5V
- R704 pad 2: /Microcontroller/REF_DIV0 -> /Microcontroller/ISP.RST
- R705 pad 1: /Microcontroller/ISP.VCC -> /Microcontroller/ISP.RST
- R705 pad 2: Net-(D601-A) -> Net-(D701-K)
- TP101 pad 1: /Measurement Unit/GATE -> /Channel Gate/CLK_REF
- TP102 pad 1: /Power Supply/PWR -> /Power Supply/BAT+
- U201 pad 1: /Frontend/CLK -> /Channel Gate/CLK_A
- U201 pad 3: Net-(D203-K) -> Net-(U201-+)
- U201 pad 4: GND -> /Frontend/VREF
- U303 pad 5: /Measurement Unit/GATE -> /Channel Gate/CLK_REF
- U303 pad 7: +5V -> GND
- U401 pad 1: /Frontend/CLK -> /Channel Gate/CH_SEL
- U401 pad 2: /Measurement Unit/GATE -> /Channel Gate/CH_SEL
- U401 pad 3: GND -> /Channel Gate/GATE_A
- U401 pad 4: Net-(U402-C) -> GND
- U401 pad 5: +5V -> Net-(U401-Pad5)
- U402 pad 1: Net-(U402-D) -> /Channel Gate/CH_SEL
- U402 pad 2: Net-(U402-C) -> /Channel Gate/CLK_REF
- U402 pad 3: GND -> /Channel Gate/B
- U402 pad 4: Net-(U402-D) -> GND
- U402 pad 5: +5V -> /Channel Gate/GATE_B
- U403 pad 1: Net-(U402-D) -> /Channel Gate/CLK_A
- U403 pad 2: /Measurement Unit/Q0 -> /Channel Gate/GATE_A
- U403 pad 3: /Measurement Unit/CLK_DIV4 -> GND
- U403 pad 4: /Measurement Unit/Q1 -> /Channel Gate/A
- U403 pad 5: unconnected-(U403-Pad5) -> +5V
- U404 pad 1: /Measurement Unit/CLK_DIV4 -> Net-(U404-D)
- U404 pad 2: Net-(U402-D) -> /Channel Gate/A
- U404 pad 4: /Measurement Unit/CLK_DIV4 -> Net-(U404-D)
- U501 pad 10: /Measurement Unit/CLK_DIV4 -> /Channel Gate/MU_CLK
- U701 pad 1: /Microcontroller/REF_RESET -> /Microcontroller/DISP_SDA
- U701 pad 11: /Microcontroller/ISP.VCC -> +5V
- U701 pad 12: /Microcontroller/REF_DIV2 -> /Channel Gate/CH_SEL
- U701 pad 13: /Microcontroller/REF_DIV1 -> /Channel Gate/CLK_REF
- U701 pad 14: /Microcontroller/REF_DIV0 -> /Microcontroller/ISP.RST
- U701 pad 15: unconnected-(U601-PC2-Pad15) -> /Microcontroller/IO_TRIG
- U701 pad 16: /Microcontroller/ISP.SCK -> Net-(U701-PC1)
- U701 pad 17: unconnected-(U601-PC0-Pad17) -> /Microcontroller/IO_SEL
- U701 pad 18: /Microcontroller/IO_ACQ_LED -> /Microcontroller/DISP_SCL
- U701 pad 19: /Microcontroller/ISP.MISO -> /Measurement Unit/RESET
- U701 pad 2: /Measurement Unit/RESET -> /Microcontroller/~{S_LOAD}
- U701 pad 20: /Microcontroller/ISP.MOSI -> /Microcontroller/REF_RESET
- U701 pad 3: /Microcontroller/~{S_LOAD} -> /Microcontroller/S_CLK
- U701 pad 4: /Microcontroller/S_CLK -> /Microcontroller/S_DATA
- U701 pad 5: /Microcontroller/S_DATA -> /Microcontroller/IO_ACQ_LED
- U701 pad 7: /Microcontroller/IO_DIV_B -> /Microcontroller/REF_DIV2
- U701 pad 8: /Microcontroller/IO_DIV_A -> /Microcontroller/REF_DIV1
- U701 pad 9: /Microcontroller/IO_HOLD_BTN -> /Microcontroller/REF_DIV0
- Y301 pad 1: Net-(C301-Pad1) -> Net-(C302-Pad1)
Routing:
- net /Channel Gate/CH_SEL: track 0.00 -> 100.1 mm, vias 0 -> 4
- net /Channel Gate/CLK_REF: track 0.00 -> 98.9 mm, vias 0 -> 4
- net /Microcontroller/ISP.MOSI: track 67.2 -> 8.33 mm, vias 1 -> 0
- net /Microcontroller/ISP.SCK: track 67.4 -> 9.98 mm, vias 1 -> 2
- net /Microcontroller/DISP_SCL: track 0.00 -> 55.3 mm, vias 0 -> 2
- net /Microcontroller/ISP.VCC: track 49.4 -> 0.00 mm
- net /Microcontroller/DISP_SDA: track 0.00 -> 49.3 mm
- net /Microcontroller/IO_TRIG: track 0.00 -> 39.1 mm, vias 0 -> 2
- net /Microcontroller/REF_DIV0: track 74.1 -> 35.1 mm, vias 2 -> 0
- net /Microcontroller/IO_HOLD_BTN: track 36.8 -> 0.00 mm
- net +5V: track 53.3 -> 89.1 mm, vias 20 -> 29
- net /Measurement Unit/GATE: track 30.7 -> 0.00 mm
- net /Measurement Unit/CLK_DIV4: track 26.1 -> 0.00 mm
- net /Microcontroller/REF_RESET: track 24.4 -> 48.0 mm
- net /Microcontroller/IO_SEL: track 0.00 -> 23.2 mm
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- added copper zone on F.Cu, net +5V
- added copper zone on F.Cu, net Net-(C201-Pad2)
- added copper zone on F.Cu, net Net-(D209-K)
Other:
- board text added: "Channel A 10 MHz ~ 325 MHz"
- board text added: "Channel B DC ~ 10 MHz"
- board text removed: "Remove jumper before ISP"
- board text removed: "Signal Input DC - 325 MHz"
- board text removed: "注意"
