File: kicad/measurement_unit.kicad_sch (KiCad schematic)
At the start: 6 parts, among them U405 74VHC4040FT, U406 74VHC4040FT, U407 74VHC4040FT

Commit message: assign references
Parts:
- renumbered CD407 to CD501, CD409 to CD502, CD408 to CD503, U405 to U501, U407 to U502, U406 to U503
Changed lines of the file:
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@@
 		(dnp no)
 		(fields_autoplaced yes)
-		(property "Reference" "#PWR0423"
+		(property "Reference" "#PWR0507"
 			(at 46.99 93.98 0)
 			(effects
@@
 			(project "frequency_counter"
 				(path "/62339e8b-4e00-440f-8d81-4472a4f50c26/f4b454df-c822-4d38-8ba5-078288da05c0"
-					(reference "#PWR0423")
+					(reference "#PWR0507")
 					(unit 1)
 				)
@@
 		(dnp no)
 		(fields_autoplaced yes)
-		(property "Reference" "#PWR0421"
+		(property "Reference" "#PWR0505"
 			(at 46.99 31.75 0)
 			(effects
@@
 			(project "frequency_counter"
 				(path "/62339e8b-4e00-440f-8d81-4472a4f50c26/f4b454df-c822-4d38-8ba5-078288da05c0"
-					(reference "#PWR0421")
+					(reference "#PWR0505")
 					(unit 1)
 				)
@@
 		(dnp no)
 		(fields_autoplaced yes)
-		(property "Reference" "CD407"
+		(property "Reference" "CD501"
 			(at 30.48 60.9599 0)
 			(effects
@@
 			(project "frequency_counter"
 				(path "/62339e8b-4e00-440f-8d81-4472a4f50c26/f4b454df-c822-4d38-8ba5-078288da05c0"
-					(reference "CD407")
+					(reference "CD501")
 					(unit 1)
 				)
@@
 		(dnp no)
 		(fields_autoplaced yes)
-		(property "Reference" "#PWR0424"
+		(property "Reference" "#PWR0508"
 			(at 46.99 144.78 0)
 			(effects
@@
 			(project "frequency_counter"
 				(path "/62339e8b-4e00-440f-8d81-4472a4f50c26/f4b454df-c822-4d38-8ba5-078288da05c0"
-					(reference "#PWR0424")
+					(reference "#PWR0508")
 					(unit 1)
 				)
@@
 		(dnp no)
 		(fields_autoplaced yes)
-		(property "Reference" "U405"
+		(property "Reference" "U501"
 			(at 49.1333 30.48 0)
 			(effects
@@
 			(project ""
 				(path "/62339e8b-4e00-440f-8d81-4472a4f50c26/f4b454df-c822-4d38-8ba5-078288da05c0"
-					(reference "U405")
+					(reference "U501")
 					(unit 1)
 				)
@@
 		(dnp no)
 		(fields_autoplaced yes)
-		(property "Reference" "CD409"
+		(property "Reference" "CD502"
 			(at 31.75 123.1899 0)
 			(effects
@@
 			(project "frequency_counter"
 				(path "/62339e8b-4e00-440f-8d81-4472a4f50c26/f4b454df-c822-4d38-8ba5-078288da05c0"
-					(reference "CD409")
+					(reference "CD502")
 					(unit 1)
 				)
@@
 		(dnp no)
 		(fields_autoplaced yes)
-		(property "Reference" "#PWR0419"
+		(property "Reference" "#PWR0503"
 			(at 27.94 121.92 0)
 			(effects
@@
 			(project "frequency_counter"
 				(path "/62339e8b-4e00-440f-8d81-4472a4f50c26/f4b454df-c822-4d38-8ba5-078288da05c0"
-					(reference "#PWR0419")
+					(reference "#PWR0503")
 					(unit 1)
 				)
@@
 		(dnp no)
 		(fields_autoplaced yes)
-		(property "Reference" "#PWR0427"
+		(property "Reference" "#PWR0511"
 			(at 99.06 31.75 0)
 			(effects
@@
 			(project "frequency_counter"
 				(path "/62339e8b-4e00-440f-8d81-4472a4f50c26/f4b454df-c822-4d38-8ba5-078288da05c0"
-					(reference "#PWR0427")
+					(reference "#PWR0511")
 					(unit 1)
 				)
@@
 		(dnp no)
 		(fields_autoplaced yes)
-		(property "Reference" "U406"
+		(property "Reference" "U503"
 			(at 101.2033 30.48 0)
 			(effects
@@
 			(project "frequency_counter"
 				(path "/62339e8b-4e00-440f-8d81-4472a4f50c26/f4b454df-c822-4d38-8ba5-078288da05c0"
-					(reference "U406")
+					(reference "U503")
 					(unit 1)
 				)
@@
 		(dnp no)
 		(fields_autoplaced yes)
-		(property "Reference" "U407"
+		(property "Reference" "U502"
 			(at 49.1333 92.71 0)
 			(effects
@@
 			(project "frequency_counter"
 				(path "/62339e8b-4e00-440f-8d81-4472a4f50c26/f4b454df-c822-4d38-8ba5-078288da05c0"
-					(reference "U407")
+					(reference "U502")
 					(unit 1)
 				)
@@
 		(dnp no)
 		(fields_autoplaced yes)
-		(property "Reference" "#PWR0428"
+		(property "Reference" "#PWR0512"
 			(at 99.06 82.55 0)
 			(effects
@@
 			(project "frequency_counter"
 				(path "/62339e8b-4e00-440f-8d81-4472a4f50c26/f4b454df-c822-4d38-8ba5-078288da05c0"
-					(reference "#PWR0428")
+					(reference "#PWR0512")
 					(unit 1)
 				)
@@
 		(on_board yes)
 		(dnp no)
-		(property "Reference" "#PWR0420"
+		(property "Reference" "#PWR0504"
 			(at 27.94 137.16 0)
 			(effects
@@
 			(project "frequency_counter"
 				(path "/62339e8b-4e00-440f-8d81-4472a4f50c26/f4b454df-c822-4d38-8ba5-078288da05c0"
-					(reference "#PWR0420")
+					(reference "#PWR0504")
 					(unit 1)
 				)
@@
 		(dnp no)
 		(fields_autoplaced yes)
-		(property "Reference" "CD408"
+		(property "Reference" "CD503"
 			(at 82.55 62.2299 0)
 			(effects
@@
 			(project "frequency_counter"
 				(path "/62339e8b-4e00-440f-8d81-4472a4f50c26/f4b454df-c822-4d38-8ba5-078288da05c0"
-					(reference "CD408")
+					(reference "CD503")
 					(unit 1)
 				)
@@
 		(on_board yes)
 		(dnp no)
-		(property "Reference" "#PWR0418"
+		(property "Reference" "#PWR0502"
 			(at 26.67 74.93 0)
 			(effects
@@
 			(project "frequency_counter"
 				(path "/62339e8b-4e00-440f-8d81-4472a4f50c26/f4b454df-c822-4d38-8ba5-078288da05c0"
-					(reference "#PWR0418")
+					(reference "#PWR0502")
 					(unit 1)
 				)
@@
 		(dnp no)
 		(fields_autoplaced yes)
-		(property "Reference" "#PWR0425"
+		(property "Reference" "#PWR0509"
 			(at 78.74 60.96 0)
 			(effects
@@
 			(project "frequency_counter"
 				(path "/62339e8b-4e00-440f-8d81-4472a4f50c26/f4b454df-c822-4d38-8ba5-078288da05c0"
-					(reference "#PWR0425")
+					(reference "#PWR0509")
 					(unit 1)
 				)
@@
 		(on_board yes)
 		(dnp no)
-		(property "Reference" "#PWR0426"
+		(property "Reference" "#PWR0510"
 			(at 78.74 76.2 0)
 			(effects
@@
 			(project "frequency_counter"
 				(path "/62339e8b-4e00-440f-8d81-4472a4f50c26/f4b454df-c822-4d38-8ba5-078288da05c0"
-					(reference "#PWR0426")
+					(reference "#PWR0510")
 					(unit 1)
 				)
@@
 		(dnp no)
 		(fields_autoplaced yes)
-		(property "Reference" "#PWR0422"
+		(property "Reference" "#PWR0506"
 			(at 46.99 82.55 0)
 			(effects
@@
 			(project "frequency_counter"
 				(path "/62339e8b-4e00-440f-8d81-4472a4f50c26/f4b454df-c822-4d38-8ba5-078288da05c0"
-					(reference "#PWR0422")
+					(reference "#PWR0506")
 					(unit 1)
 				)
@@
 		(dnp no)
 		(fields_autoplaced yes)
-		(property "Reference" "#PWR0417"
+		(property "Reference" "#PWR0501"
 			(at 26.67 59.69 0)
 			(effects
@@
 			(project "frequency_counter"
 				(path "/62339e8b-4e00-440f-8d81-4472a4f50c26/f4b454df-c822-4d38-8ba5-078288da05c0"
-					(reference "#PWR0417")
-					(unit 1)
-				)
+					(reference "#PWR0501")
+					(unit 1)
+				)

Commit message: redesign pcb for 2.0
Parts:
- renumbered U503 to U502, U502 to U503
Changed lines of the file:
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@@
 		(dnp no)
 		(fields_autoplaced yes)
-		(property "Reference" "U503"
+		(property "Reference" "U502"
 			(at 101.2033 30.48 0)
 			(effects
@@
 			(project "frequency_counter"
 				(path "/62339e8b-4e00-440f-8d81-4472a4f50c26/f4b454df-c822-4d38-8ba5-078288da05c0"
-					(reference "U503")
+					(reference "U502")
 					(unit 1)
 				)
@@
 		(dnp no)
 		(fields_autoplaced yes)
-		(property "Reference" "U502"
+		(property "Reference" "U503"
 			(at 49.1333 92.71 0)
 			(effects
@@
 			(project "frequency_counter"
 				(path "/62339e8b-4e00-440f-8d81-4472a4f50c26/f4b454df-c822-4d38-8ba5-078288da05c0"
-					(reference "U502")
+					(reference "U503")
 					(unit 1)
 				)
