File: kicad/power_supply.kicad_sch (KiCad schematic)
At the start: 27 parts, among them Q801 SIL2300, U801 TP4057, U802 DW01, U803 LM4040D25FTA, U804 MCP6001, U805 TPS613222ADBV

Commit message: redesign pcb for 2.0
Parts:
- removed CD803: 0.1uF, Custom:C_0402_1005Metric_Fix, symbol Device:C
- renumbered R807 to R806, R808 to R807, R806 to R808, U805 to U803, U803 to U804, U804 to U805
Changed lines of the file:
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@@
 	)
 	(junction
-		(at 166.37 104.14)
-		(diameter 0)
-		(color 0 0 0 0)
-	)
-	(junction
 		(at 66.04 110.49)
 		(diameter 0)
@@
 	(wire
 		(pts
-			(xy 158.75 104.14) (xy 166.37 104.14)
+			(xy 158.75 104.14) (xy 161.29 104.14)
 		)
 		(stroke
@@
 	(wire
 		(pts
-			(xy 166.37 104.14) (xy 166.37 106.68)
-		)
-		(stroke
-			(width 0)
-			(type default)
-		)
-	)
-	(wire
-		(pts
 			(xy 146.05 45.72) (xy 146.05 59.69)
 		)
@@
 	(wire
 		(pts
-			(xy 166.37 114.3) (xy 166.37 116.84)
-		)
-		(stroke
-			(width 0)
-			(type default)
-		)
-	)
-	(wire
-		(pts
 			(xy 82.55 41.91) (xy 82.55 24.13)
 		)
@@
 	(wire
 		(pts
-			(xy 166.37 104.14) (xy 168.91 104.14)
-		)
-		(stroke
-			(width 0)
-			(type default)
-		)
-	)
-	(wire
-		(pts
 			(xy 95.25 62.23) (xy 95.25 64.77)
 		)
@@
 	(hierarchical_label "REF_2V5"
 		(shape passive)
-		(at 168.91 104.14 0)
+		(at 161.29 104.14 0)
 		(effects
 			(font
@@
 		(dnp no)
 		(fields_autoplaced yes)
-		(property "Reference" "#PWR0810"
+		(property "Reference" "#PWR0114"
 			(at 119.38 92.71 0)
 			(effects
@@
 			(project ""
 				(path "/62339e8b-4e00-440f-8d81-4472a4f50c26/713bd15e-856e-443f-a6a5-b9988a9adf89"
-					(reference "#PWR0810")
+					(reference "#PWR0114")
 					(unit 1)
 				)
@@
 		(dnp no)
 		(fields_autoplaced yes)
-		(property "Reference" "R807"
+		(property "Reference" "R806"
 			(at 49.53 80.01 90)
 			(effects
@@
 			(project ""
 				(path "/62339e8b-4e00-440f-8d81-4472a4f50c26/713bd15e-856e-443f-a6a5-b9988a9adf89"
-					(reference "R807")
+					(reference "R806")
 					(unit 1)
 				)
@@
 		(dnp no)
 		(fields_autoplaced yes)
-		(property "Reference" "#FLG0801"
+		(property "Reference" "#FLG0101"
 			(at 36.195 86.36 0)
 			(effects
@@
 			(project "frequency_counter"
 				(path "/62339e8b-4e00-440f-8d81-4472a4f50c26/713bd15e-856e-443f-a6a5-b9988a9adf89"
-					(reference "#FLG0801")
+					(reference "#FLG0101")
 					(unit 1)
 				)
@@
 		(dnp no)
 		(fields_autoplaced yes)
-		(property "Reference" "#PWR0803"
+		(property "Reference" "#PWR0124"
 			(at 66.04 129.54 0)
 			(effects
@@
 			(project "frequency_counter"
 				(path "/62339e8b-4e00-440f-8d81-4472a4f50c26/713bd15e-856e-443f-a6a5-b9988a9adf89"
-					(reference "#PWR0803")
-					(unit 1)
-				)
-			)
-		)
-	)
-	(symbol
-		(lib_id "power:GND")
-		(at 166.37 116.84 0)
-		(unit 1)
-		(exclude_from_sim no)
-		(in_bom yes)
-		(on_board yes)
-		(dnp no)
-		(fields_autoplaced yes)
-		(property "Reference" "#PWR0815"
-			(at 166.37 123.19 0)
-			(effects
-				(font
-					(size 1.27 1.27)
-				)
-				(hide yes)
-			)
-		)
-		(property "Value" "GND"
-			(at 166.37 121.92 0)
-			(effects
-				(font
-					(size 1.27 1.27)
-				)
-			)
-		)
-		(property "Footprint" ""
-			(at 166.37 116.84 0)
-			(effects
-				(font
-					(size 1.27 1.27)
-				)
-				(hide yes)
-			)
-		)
-		(property "Datasheet" ""
-			(at 166.37 116.84 0)
-			(effects
-				(font
-					(size 1.27 1.27)
-				)
-				(hide yes)
-			)
-		)
-		(property "Description" "Power symbol creates a global label with name \"GND\" , ground"
-			(at 166.37 116.84 0)
-			(effects
-				(font
-					(size 1.27 1.27)
-				)
-				(hide yes)
-			)
-		)
-		(pin "1"
-		)
-		(instances
-			(project "frequency_counter"
-				(path "/62339e8b-4e00-440f-8d81-4472a4f50c26/713bd15e-856e-443f-a6a5-b9988a9adf89"
-					(reference "#PWR0815")
+					(reference "#PWR0124")
 					(unit 1)
 				)
@@
 		(dnp no)
 		(fields_autoplaced yes)
-		(property "Reference" "#PWR0805"
+		(property "Reference" "#PWR0122"
 			(at 80.01 129.54 0)
 			(effects
@@
 			(project "frequency_counter"
 				(path "/62339e8b-4e00-440f-8d81-4472a4f50c26/713bd15e-856e-443f-a6a5-b9988a9adf89"
-					(reference "#PWR0805")
+					(reference "#PWR0122")
 					(unit 1)
 				)
@@
 		(dnp no)
 		(fields_autoplaced yes)
-		(property "Reference" "R808"
+		(property "Reference" "R807"
 			(at 91.44 104.14 90)
 			(effects
@@
 			(project "frequency_counter"
 				(path "/62339e8b-4e00-440f-8d81-4472a4f50c26/713bd15e-856e-443f-a6a5-b9988a9adf89"
-					(reference "R808")
+					(reference "R807")
 					(unit 1)
 				)
@@
 		(dnp no)
 		(fields_autoplaced yes)
-		(property "Reference" "U803"
+		(property "Reference" "U804"
 			(at 121.92 106.6799 90)
 			(effects
@@
 			(project ""
 				(path "/62339e8b-4e00-440f-8d81-4472a4f50c26/713bd15e-856e-443f-a6a5-b9988a9adf89"
-					(reference "U803")
+					(reference "U804")
 					(unit 1)
 				)
@@
 	)
 	(symbol
-		(lib_id "Device:C")
-		(at 166.37 110.49 0)
-		(unit 1)
-		(exclude_from_sim no)
-		(in_bom yes)
-		(on_board yes)
-		(dnp no)
-		(fields_autoplaced yes)
-		(property "Reference" "CD803"
-			(at 170.18 109.2199 0)
-			(effects
-				(font
-					(size 1.27 1.27)
-				)
-				(justify left)
-			)
-		)
-		(property "Value" "0.1uF"
-			(at 170.18 111.7599 0)
-			(effects
-				(font
-					(size 1.27 1.27)
-				)
-				(justify left)
-			)
-		)
-		(property "Footprint" "Custom:C_0402_1005Metric_Fix"
-			(at 167.3352 114.3 0)
-			(effects
-				(font
-					(size 1.27 1.27)
-				)
-				(hide yes)
-			)
-		)
-		(property "Datasheet" "~"
-			(at 166.37 110.49 0)
-			(effects
-				(font
-					(size 1.27 1.27)
-				)
-				(hide yes)
-			)
-		)
-		(property "Description" "Unpolarized capacitor"
-			(at 166.37 110.49 0)
-			(effects
-				(font
-					(size 1.27 1.27)
-				)
-				(hide yes)
-			)
-		)
-		(property "MPN" "KGM05AR51C104KH"
-			(at 166.37 110.49 0)
-			(effects
-				(font
-					(size 1.27 1.27)
-				)
-				(hide yes)
-			)
-		)
-		(pin "2"
-		)
-		(pin "1"
-		)
-		(instances
-			(project "frequency_counter"
-				(path "/62339e8b-4e00-440f-8d81-4472a4f50c26/713bd15e-856e-443f-a6a5-b9988a9adf89"
-					(reference "CD803")
-					(unit 1)
-				)
-			)
-		)
-	)
-	(symbol
 		(lib_id "Battery_Management:DW01A")
 		(at 170.18 35.56 0)
@@
 		(dnp no)
 		(fields_autoplaced yes)
-		(property "Reference" "#PWR0804"
+		(property "Reference" "#PWR0123"
 			(at 80.01 111.76 0)
 			(effects
@@
 			(project "frequency_counter"
 				(path "/62339e8b-4e00-440f-8d81-4472a4f50c26/713bd15e-856e-443f-a6a5-b9988a9adf89"
-					(reference "#PWR0804")
+					(reference "#PWR0123")
 					(unit 1)
 				)
@@
 		(dnp no)
 		(fields_autoplaced yes)
-		(property "Reference" "#PWR0811"
+		(property "Reference" "#PWR0115"
 			(at 119.38 120.65 0)
 			(effects
@@
 			(project ""
 				(path "/62339e8b-4e00-440f-8d81-4472a4f50c26/713bd15e-856e-443f-a6a5-b9988a9adf89"
-					(reference "#PWR0811")
+					(reference "#PWR0115")
 					(unit 1)
 				)
@@
 		(dnp no)
 		(fields_autoplaced yes)
-		(property "Reference" "#PWR0808"
+		(property "Reference" "#PWR0121"
 			(at 99.06 129.54 0)
 			(effects
@@
 			(project "frequency_counter"
 				(path "/62339e8b-4e00-440f-8d81-4472a4f50c26/713bd15e-856e-443f-a6a5-b9988a9adf89"
-					(reference "#PWR0808")
+					(reference "#PWR0121")
 					(unit 1)
 				)
@@
 		(on_board yes)
 		(dnp no)
-		(property "Reference" "U804"
+		(property "Reference" "U805"
 			(at 152.146 108.204 0)
 			(effects
@@
 			(project ""
 				(path "/62339e8b-4e00-440f-8d81-4472a4f50c26/713bd15e-856e-443f-a6a5-b9988a9adf89"
-					(reference "U804")
+					(reference "U805")
 					(unit 1)
 				)
@@
 		(dnp no)
 		(fields_autoplaced yes)
-		(property "Reference" "#PWR0802"
+		(property "Reference" "#PWR0120"
 			(at 53.34 129.54 0)
 			(effects
@@
 			(project ""
 				(path "/62339e8b-4e00-440f-8d81-4472a4f50c26/713bd15e-856e-443f-a6a5-b9988a9adf89"
-					(reference "#PWR0802")
+					(reference "#PWR0120")
 					(unit 1)
 				)
@@
 		(dnp no)
 		(fields_autoplaced yes)
-		(property "Reference" "#PWR0813"
+		(property "Reference" "#PWR0116"
 			(at 146.05 120.65 0)
 			(effects
@@
 			(project ""
 				(path "/62339e8b-4e00-440f-8d81-4472a4f50c26/713bd15e-856e-443f-a6a5-b9988a9adf89"
-					(reference "#PWR0813")
+					(reference "#PWR0116")
 					(unit 1)
 				)
@@
 		(dnp no)
 		(fields_autoplaced yes)
-		(property "Reference" "U805"
+		(property "Reference" "U803"
 			(at 53.34 102.87 0)
 			(effects
@@
 			(project ""
 				(path "/62339e8b-4e00-440f-8d81-4472a4f50c26/713bd15e-856e-443f-a6a5-b9988a9adf89"
-					(reference "U805")
+					(reference "U803")
 					(unit 1)
 				)
@@
 		(dnp no)
 		(fields_autoplaced yes)
-		(property "Reference" "#PWR0812"
+		(property "Reference" "#PWR0117"
 			(at 146.05 95.25 0)
 			(effects
@@
 			(project ""
 				(path "/62339e8b-4e00-440f-8d81-4472a4f50c26/713bd15e-856e-443f-a6a5-b9988a9adf89"
-					(reference "#PWR0812")
+					(reference "#PWR0117")
 					(unit 1)
 				)
@@
 		(dnp no)
 		(fields_autoplaced yes)
-		(property "Reference" "R806"
+		(property "Reference" "R808"
 			(at 121.92 93.9799 0)
 			(effects
@@
 			(project ""
 				(path "/62339e8b-4e00-440f-8d81-4472a4f50c26/713bd15e-856e-443f-a6a5-b9988a9adf89"
-					(reference "R806")
+					(reference "R808")
 					(unit 1)
 				)
@@
 		(dnp no)
 		(fields_autoplaced yes)
-		(property "Reference" "#PWR0814"
+		(property "Reference" "#PWR0119"
 			(at 165.1 93.98 0)
 			(effects
@@
 			(project ""
 				(path "/62339e8b-4e00-440f-8d81-4472a4f50c26/713bd15e-856e-443f-a6a5-b9988a9adf89"
-					(reference "#PWR0814")
+					(reference "#PWR0119")
 					(unit 1)
 				)
